File: kicad/test2/rectifier/rectifier.sch (KiCad schematic (older format))
At the start: 12 parts

Commit message: yes
Connections:
- new net: D?.~ (K), D?.~ (K), R1.1
Changed lines of the file:
@@
 	8500 3300 8500 3250
 Connection ~ 8500 3250
-Text GLabel 9400 2850 2    50   Input ~ 0
+Text GLabel 9400 2850 2    50   Output ~ 0
 Vdirdiff
 Wire Notes Line style dash_dot
